File: _autosave-deskdocker_v1.kicad_pcb (KiCad board)
At the start: 2 copper layers, 168.2 x 130.7 mm, 115 parts, among them J1 USB_C_Receptacle_USB2.0, J2 USB_C_Receptacle_USB2.0, J3 OLED, SW1 SW_PUSH, SW10 SW_PUSH, SW11 SW_PUSH, SW12 SW_PUSH, SW13 SW_PUSH, SW14 SW_PUSH, SW15 SW_PUSH, SW16 SW_PUSH, SW17 SW_PUSH, SW18 SW_PUSH, SW19 SW_PUSH, SW2 SW_PUSH, SW20 SW_PUSH, SW21 SW_PUSH, SW22 SW_PUSH, SW23 SW_PUSH, SW24 SW_PUSH, SW25 Rotary_Encoder_Switch, SW3 SW_PUSH, SW4 SW_PUSH, SW5 SW_PUSH, SW6 SW_PUSH, SW7 SW_PUSH, SW8 SW_PUSH, SW9 SW_PUSH, U1 ATMEGA32U4, U2 MIC5219-5.0YMM, X1 16Mhz

Commit message: init commit
Parts:
- removed the SW24 at (150.6, 110.5)
- added R6: 330, Resistor_SMD:R_0805_2012Metric, F.Cu at (151.0, 83.1)
- added R8: 330, Resistor_SMD:R_0805_2012Metric, F.Cu at (155.4, 83.1)
- added RED1: LED1, LED_SMD:LED_0603_1608Metric, F.Cu at (252.1, 64.1)
- added RED1: LED1, LED_SMD:LED_0603_1608Metric, F.Cu at (248.3, 64.1)
- SW22: moved to B.Cu
- moved SW20 192.4 mm to (93.4, 96.0)
- moved D10 190.0 mm to (227.8, 73.8)
- moved D11 190.0 mm to (238.5, 76.3)
- moved D12 190.0 mm to (219.8, 93.3)
- moved D13 190.0 mm to (226.0, 91.8)
- moved D14 190.0 mm to (217.8, 81.7)
- moved D15 190.0 mm to (220.6, 72.1)
- moved D16 190.0 mm to (238.2, 92.4)
- moved D17 190.0 mm to (243.2, 79.3)
- moved D18 190.0 mm to (219.8, 90.2)
- moved D19 190.0 mm to (232.3, 73.8)
- moved D20 190.0 mm to (234.3, 84.0)
- moved D21 190.0 mm to (219.3, 99.5)
- moved D22 190.0 mm to (225.2, 88.7)
- moved D23 190.0 mm to (217.8, 78.7)
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Connections:
- C19 pad 2: +5V -> GND
- C3 pad 2: +5V -> GND
- C6 pad 1: +3V3 -> VCC
- C7 pad 1: +3V3 -> VCC
- C8 pad 1: +3V3 -> VCC
- JP1 pad 2: +3V3 -> VCC
- R1 pad 1: +3V3 -> VCC
- U2 pad 3: +3V3 -> VCC
Routing:
- net (no net): vias 1 -> 0
Other:
- board size 168.2 x 130.7 mm -> 112.6 x 70.4 mm
