File: deskdocker_v1.kicad_pcb (KiCad board)
At the start: 2 copper layers, 421.6 x 211.2 mm, 113 parts, among them J1 USB_C_Receptacle_USB2.0, J2 USB_C_Receptacle_USB2.0, SW1 SW_PUSH, SW10 SW_PUSH, SW11 SW_PUSH, SW12 SW_PUSH, SW13 SW_PUSH, SW14 SW_PUSH, SW15 SW_PUSH, SW16 SW_PUSH, SW17 SW_PUSH, SW18 SW_PUSH, SW19 SW_PUSH, SW2 SW_PUSH, SW20 SW_PUSH, SW21 SW_PUSH, SW22 SW_PUSH, SW23 SW_PUSH, SW24 SW_PUSH, SW25 Rotary_Encoder_Switch, SW3 SW_PUSH, SW4 SW_PUSH, SW5 SW_PUSH, SW6 SW_PUSH, SW7 SW_PUSH, SW8 SW_PUSH, SW9 SW_PUSH, U1 ATMEGA32U4, U2 MIC5219-5.0YMM, X1 16Mhz

Commit message: init commit
Parts:
- added J3: OLED, Display:Generic_0.96in-128x64-OLED-Display-IIC, F.Cu at (147.3, 39.8)
- added RED1: LED1, LED_SMD:LED_0603_1608Metric, F.Cu at (167.5, 56.7)
- added RED1: LED1, LED_SMD:LED_0603_1608Metric, F.Cu at (163.8, 56.7)
- J1, J2: footprint Connector_USB:USB_C_Receptacle_GCT_USB4085 -> Connector_USB:USB_C_Receptacle_HRO_TYPE-C-31-M-12
- moved D16 296.0 mm to (50.8, 123.7)
- moved D15 210.6 mm to (33.2, 103.3)
- moved D8 210.6 mm to (37.6, 100.4)
- moved D24 202.5 mm to (42.1, 130.3)
- moved D10 195.6 mm to (40.4, 105.0)
- moved D19 195.6 mm to (44.9, 105.0)
- moved C6 195.3 mm to (43.3, 24.9)
- moved D21 192.5 mm to (31.9, 130.7)
- moved D14 190.9 mm to (30.4, 113.0)
- moved D23 190.9 mm to (30.4, 109.9)
- moved D4 190.9 mm to (25.7, 121.1)
- moved D9 190.9 mm to (25.7, 118.0)
- moved D12 190.7 mm to (32.4, 124.5)
- moved D18 190.7 mm to (32.4, 121.4)
- moved C1 186.8 mm to (36.9, 25.2)
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Connections:
- C6 pad 1: VCC -> +3V3
- C7 pad 1: VCC -> +3V3
- C8 pad 1: VCC -> +3V3
- D1 pad 1: ROW0 -> A3
- D10 pad 1: ROW1 -> A2
- D11 pad 1: ROW1 -> A2
- D12 pad 1: ROW1 -> A2
- D13 pad 1: ROW2 -> A1
- D14 pad 1: ROW2 -> A1
- D15 pad 1: ROW2 -> A1
- D16 pad 1: ROW2 -> A1
- D17 pad 1: ROW2 -> A1
- D18 pad 1: ROW2 -> A1
- D19 pad 1: ROW3 -> A0
- D2 pad 1: ROW0 -> A3
- D20 pad 1: ROW3 -> A0
- D21 pad 1: ROW3 -> A0
- D22 pad 1: ROW3 -> A0
- D23 pad 1: ROW3 -> A0
- D24 pad 1: ROW3 -> A0
- D3 pad 1: ROW0 -> A3
- D4 pad 1: ROW0 -> A3
- D5 pad 1: ROW0 -> A3
- D6 pad 1: ROW0 -> A3
- D7 pad 1: ROW1 -> A2
- D8 pad 1: ROW1 -> A2
- D9 pad 1: ROW1 -> A2
- JP1 pad 2: VCC -> +3V3
- R1 pad 1: VCC -> +3V3
- R2 pad 1: +3V3 -> VCC
- U2 pad 3: VCC -> +3V3
Other:
- board size 421.6 x 211.2 mm -> 168.2 x 130.7 mm

Commit message: schematic done -ish?
Parts:
- removed the RED1 at (167.5, 56.7)
- removed the RED1 at (163.8, 56.7)
- added R6: 330, Resistor_SMD:R_0805_2012Metric, F.Cu at (151.0, 83.1)
- added R8: 330, Resistor_SMD:R_0805_2012Metric, F.Cu at (155.4, 83.1)
- added RED1: LED1, LED_SMD:LED_0603_1608Metric, F.Cu at (252.1, 64.1)
- added RED1: LED1, LED_SMD:LED_0603_1608Metric, F.Cu at (248.3, 64.1)
- SW22: moved to B.Cu
- moved SW20 192.4 mm to (93.4, 96.0)
- moved D10 190.0 mm to (227.8, 73.8)
- moved D11 190.0 mm to (238.5, 76.3)
- moved D12 190.0 mm to (219.8, 93.3)
- moved D13 190.0 mm to (226.0, 91.8)
- moved D14 190.0 mm to (217.8, 81.7)
- moved D15 190.0 mm to (220.6, 72.1)
- moved D16 190.0 mm to (238.2, 92.4)
- moved D17 190.0 mm to (243.2, 79.3)
- moved D18 190.0 mm to (219.8, 90.2)
- moved D19 190.0 mm to (232.3, 73.8)
- moved D20 190.0 mm to (234.3, 84.0)
- moved D21 190.0 mm to (219.3, 99.5)
- moved D22 190.0 mm to (225.2, 88.7)
- moved D23 190.0 mm to (217.8, 78.7)
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Connections:
- C1 pad 1: +5V -> GND
- C19 pad 2: +5V -> GND
- C2 pad 2: +5V -> GND
- C3 pad 2: +5V -> GND
- C4 pad 2: +5V -> GND
- C5 pad 2: +5V -> GND
- C6 pad 1: +3V3 -> VCC
- C6 pad 2: +5V -> GND
- C7 pad 1: +3V3 -> VCC
- C7 pad 2: +5V -> GND
- C8 pad 1: +3V3 -> VCC
- C8 pad 2: +5V -> GND
- J1 pad A1: +5V -> GND
- J1 pad A12: +5V -> GND
- J1 pad B1: +5V -> GND
- J1 pad B12: +5V -> GND
- J1 pad S1: +5V -> GND
- J3 pad 1: +5V -> GND
- JP1 pad 2: +3V3 -> VCC
- L1 pad 2: +5V -> GND
- L15 pad 2: +5V -> GND
- L16 pad 2: +5V -> GND
- L17 pad 2: +5V -> GND
- L18 pad 2: +5V -> GND
- L19 pad 2: +5V -> GND
- L2 pad 2: +5V -> GND
- L20 pad 2: +5V -> GND
- L21 pad 2: +5V -> GND
- L22 pad 2: +5V -> GND
- L23 pad 2: +5V -> GND
- L24 pad 2: +5V -> GND
- L25 pad 2: +5V -> GND
- L26 pad 2: +5V -> GND
- L27 pad 2: +5V -> GND
- L28 pad 2: +5V -> GND
- L29 pad 2: +5V -> GND
- L3 pad 2: +5V -> GND
- L30 pad 2: +5V -> GND
- L31 pad 2: +5V -> GND
- L32 pad 2: +5V -> GND
- L4 pad 2: +5V -> GND
- L5 pad 2: +5V -> GND
- L6 pad 2: +5V -> GND
- L7 pad 2: +5V -> GND
- L8 pad 2: +5V -> GND
- R1 pad 1: +3V3 -> VCC
- RED1 pad 1: +5V -> GND
- RESET_SW1 pad 2: +5V -> GND
- U1 pad 15: +5V -> GND
- U1 pad 23: +5V -> GND
- U1 pad 33: +5V -> GND
- U1 pad 35: +5V -> GND
- U1 pad 43: +5V -> GND
- U1 pad 5: +5V -> GND
- U2 pad 3: +3V3 -> VCC
- U2 pad 5: +5V -> GND
- U2 pad 6: +5V -> GND
- U2 pad 7: +5V -> GND
- U2 pad 8: +5V -> GND
Other:
- board size 168.2 x 130.7 mm -> 112.6 x 70.4 mm

Commit message: schematic pre-final
Parts:
- removed the RED1 at (252.1, 64.1)
- removed the RED1 at (248.3, 64.1)
- removed the SW19 at (74.4, 96.0)
- added R10: 330, Resistor_SMD:R_0805_2012Metric, F.Cu at (-488.5, 65.5)
- added R11: 5.1k, Resistor_SMD:R_0805_2012Metric, F.Cu at (195.8, 71.2)
- added R12: 5.1k, Resistor_SMD:R_0805_2012Metric, F.Cu at (200.2, 71.2)
- added R9: 330, Resistor_SMD:R_0805_2012Metric, F.Cu at (-492.9, 65.5)
- added RED1: LED1, LED_SMD:LED_0603_1608Metric, F.Cu at (151.8, 56.1)
- added RED1: LED1, LED_SMD:LED_0603_1608Metric, F.Cu at (155.6, 56.1)
- added RED1: LED1, LED_SMD:LED_0603_1608Metric, F.Cu at (147.8, 56.1)
- added RED1: LED1, LED_SMD:LED_0603_1608Metric, F.Cu at (143.9, 56.1)
- moved R4 122.3 mm to (36.4, 25.1), turned to 90 degrees
- moved R7 120.0 mm to (46.7, 25.1), turned to 90 degrees
- moved R3 115.2 mm to (40.0, 25.0), turned to 90 degrees
- moved R5 106.5 mm to (43.7, 25.1), turned to 90 degrees
- moved RED1 104.7 mm to (140.2, 56.1)
- moved C1 72.3 mm to (107.7, 10.3)
- moved C6 72.3 mm to (114.1, 10.0)
- moved L3 34.3 mm to (228.0, 21.1)
- moved L2 22.0 mm to (221.2, 21.1)
- moved L8 18.6 mm to (193.9, 14.0)
- moved C5 17.8 mm to (53.2, 10.6)
- moved F1 6.17 mm to (134.8, 61.9)
- moved U1 2.44 mm to (147.7, 67.1)
- moved X1 2.19 mm to (156.3, 74.5)
- moved R2 2.07 mm to (148.1, 79.0)
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- renumbered SW25 to SW19
Connections:
- J2 pad A1: Net-(J2-PadA1) -> GND
- J2 pad A12: Net-(J2-PadA1) -> GND
- J2 pad A4: Net-(J2-PadA4) -> VCC
- J2 pad A9: Net-(J2-PadA4) -> VCC
- J2 pad B1: Net-(J2-PadA1) -> GND
- J2 pad B12: Net-(J2-PadA1) -> GND
- J2 pad B4: Net-(J2-PadA4) -> VCC
- J2 pad B7: Net-(J2-PadB7) -> RX
- J2 pad B9: Net-(J2-PadA4) -> VCC
- J2 pad S1: Net-(J2-PadS1) -> GND
- J3 pad 3: SCL -> D3
- J3 pad 4: SDA -> D2
- L1 pad 3: LED -> D9
- L9 pad 3: Net-(L8-Pad1) -> D10
- SW19 pad A: Net-(SW25-PadA) -> A4
- SW19 pad B: Net-(SW25-PadB) -> A5
- SW19 pad C: Net-(SW25-PadC) -> GND
- SW19 pad S1: Net-(SW25-PadS1) -> Net-(D19-Pad2)
- SW19 pad S2: Net-(SW25-PadS2) -> COL0
- U1 pad 1: D7 -> COL3
- U1 pad 25: D4 -> COL0
- U1 pad 27: D6 -> COL2
- U1 pad 28: D8 -> COL4
- U1 pad 31: D5 -> COL1
- U1 pad 40: Net-(U1-Pad40) -> A4
- U1 pad 41: Net-(U1-Pad41) -> A5
Other:
- board size 112.6 x 70.4 mm -> 150.7 x 107.2 mm
- net class Power added: clearance 0.2, trace_width 0.25, via_dia 0.8, via_drill 0.4

Commit message: schematic final_1
Parts:
- removed L32: SK6812_mini, keebio_parts:SK6812-MINI-E
- removed the RED1 at (151.8, 56.1)
- removed the RED1 at (155.6, 56.1)
- removed the RED1 at (147.8, 56.1)
- removed the RED1 at (143.9, 56.1)
- removed the RED1 at (140.2, 56.1)
- added D26: Green, LED_SMD:LED_0603_1608Metric, F.Cu at (143.4, 55.1)
- added D27: Orange, LED_SMD:LED_0603_1608Metric, F.Cu at (151.1, 55.2)
- added D28: Blue, LED_SMD:LED_0603_1608Metric, F.Cu at (147.5, 55.1)
- added D29: Yellow, LED_SMD:LED_0603_1608Metric, F.Cu at (155.2, 55.2)
- added L33: WS2812_LED, keebio_parts:WS2812B, B.Cu at (163.1, 112.2)
- added L34: WS2812_LED, keebio_parts:WS2812B, B.Cu at (102.6, 88.5)
- added L35: WS2812_LED, keebio_parts:WS2812B, B.Cu at (72.5, 80.8)
- added L36: WS2812_LED, keebio_parts:WS2812B, B.Cu at (33.8, 72.2)
- added RED1: LED1, LED_SMD:LED_0603_1608Metric, F.Cu at (139.6, 55.0)
- added REF**: SW_Cherry_MX_2.00u_Vertical_PCB, Button_Switch_Keyboard:SW_Cherry_MX_2.00u_Vertical_PCB, F.Cu at (149.8, 110.4)
- added REF**: SW_Cherry_MX_2.00u_Vertical_PCB, Button_Switch_Keyboard:SW_Cherry_MX_2.00u_Vertical_PCB, F.Cu at (131.4, 105.5)
- L1, L10, L11, L12, L13, L14, L15, L16, L17, L18, L19, L2, L20, L21, L22, L23, L24, L25, L26, L27, L28, L29, L3, L30, L31, L4, L5, L6, L7, L8, L9: moved to B.Cu
- SW22: moved to F.Cu
- SW23, SW24: footprint keebio_parts:MX-Alps_Switch_Cutout-1u_2u -> keyswitches:Kailh_socket_MX
- moved R10 647.3 mm to (158.8, 59.9)
- moved R9 647.3 mm to (154.3, 59.9)
- moved L15 252.2 mm to (24.2, 54.0)
- moved L9 227.2 mm to (24.2, 35.0)
- moved L21 224.3 mm to (24.2, 73.0)
- moved L10 224.1 mm to (43.2, 33.0)
- moved L23 222.1 mm to (62.2, 59.0)
- moved L22 219.4 mm to (43.2, 71.0)
- moved L27 210.3 mm to (93.4, 88.5)
- moved L16 209.3 mm to (43.2, 52.0)
- moved L12 208.6 mm to (81.2, 18.0)
- moved D7 207.9 mm to (32.4, 58.5), turned to 90 degrees
- moved L11 196.5 mm to (62.2, 21.0)
- moved D13 194.1 mm to (32.4, 77.5), turned to 90 degrees
- moved L18 185.8 mm to (81.2, 37.0)
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Connections:
- J2 pad A5: Net-(J2-PadA5) -> +5V
- J2 pad A6: Net-(J2-PadA6) -> RX
- J2 pad B5: Net-(J2-PadB5) -> +5V
- U1 pad 26: Net-(U1-Pad26) -> COL2
- U1 pad 27: COL2 -> Net-(R9-Pad1)
- U1 pad 32: Net-(U1-Pad32) -> Net-(R10-Pad1)
Other:
- board size 150.7 x 107.2 mm -> 169.4 x 122.6 mm

Commit message: schematic final_2
Parts:
- added H2: Hole, MountingHole:MountingHole_2.2mm_M2, F.Cu at (155.9, 87.1)
- added Kailh PG1350: Choc, keebio_parts:Kailh-PG1350-1.5u, F.Cu at (160.5, 115.0)
- added r: SW_Push_1P1T_NO_6x6mm_H9.5mm, Button_Switch_SMD:SW_Push_1P1T_NO_6x6mm_H9.5mm, F.Cu at (108.1, 20.0)
- added r: SW_Push_1P1T_NO_6x6mm_H9.5mm, Button_Switch_SMD:SW_Push_1P1T_NO_6x6mm_H9.5mm, F.Cu at (97.3, 20.0)
- SW19: value Rotary_Encoder_Switch -> Rotary_Encoder
- moved L33 192.7 mm to (-19.2, 49.8)
- moved L6 162.1 mm to (-6.50, 82.5)
- moved L5 154.6 mm to (4.95, 28.4)
- moved L1 154.4 mm to (4.30, 63.3)
- moved L7 143.5 mm to (5.30, 39.5)
- moved L2 117.7 mm to (-8.40, 31.8)
- moved U2 111.2 mm to (34.0, 29.7)
- moved SW19 109.2 mm to (64.8, 90.8), turned to 0 degrees
- moved L34 106.5 mm to (1.85, 54.1)
- moved H4 97.1 mm to (132.1, 82.8)
- moved D24 95.0 mm to (134.8, 106.3), turned to 260 degrees
- moved D23 89.5 mm to (131.9, 104.0), turned to 80 degrees
- moved C19 83.5 mm to (190.1, 79.6)
- moved C3 83.5 mm to (194.4, 91.0)
- moved C7 83.5 mm to (199.8, 84.2)
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Routing:
- net Net-(L28-Pad1): vias 0 -> 2
Other:
- board size 169.4 x 122.6 mm -> 159.6 x 117 mm
- board text added: "endless v1.0"

Commit message: schematic final_3
Parts:
- removed D27: Orange, LED_SMD:LED_0603_1608Metric
- removed the REF** at (178.7, 55.1)
- removed the RESET_SW1 at (155.9, 0.49)
- removed r (x2): SW_Push_1P1T_NO_6x6mm_H9.5mm, Button_Switch_SMD:SW_Push_1P1T_NO_6x6mm_H9.5mm
- added BZ1: Buzzer, Buzzer_Beeper:MagneticBuzzer_PUI_AT-0927-TT-6-R, F.Cu at (141.5, 73.7)
- added L2: WS2812_LED, keebio_parts:WS2812B, F.Cu at (52.1, -27.9)
- added L32: SK6812_mini, keebio_parts:SK6812-MINI-E, F.Cu at (64.6, 77.2)
- added L5: WS2812_LED, keebio_parts:WS2812B, F.Cu at (19.4, 22.9)
- added L7: WS2812_LED, keebio_parts:WS2812B, F.Cu at (47.4, 22.8)
- added L7: WS2812_LED, keebio_parts:WS2812B, F.Cu at (33.2, 23.1)
- added REF**: MagneticBuzzer_PUI_AT-0927-TT-6-R, Buzzer_Beeper:MagneticBuzzer_PUI_AT-0927-TT-6-R, F.Cu at (149.6, -8.15)
- added RESET_SW1: SW_PUSH, Button_Switch_SMD:SW_Push_1P1T_NO_6x6mm_H9.5mm, F.Cu at (177.1, 14.9)
- added RESET_SW1: SW_PUSH, Button_Switch_SMD:SW_Push_1P1T_NO_6x6mm_H9.5mm, F.Cu at (194.9, 12.9)
- D26, D28, D29, RED1: footprint LED_SMD:LED_0603_1608Metric -> LED_THT:LED_D3.0mm
- J1, J2: footprint Connector_USB:USB_C_Receptacle_HRO_TYPE-C-31-M-12 -> private:USB_C_TH_6pin
- moved D28 127.8 mm to (31.8, -5.30)
- moved L3 101.8 mm to (-22.8, 61.5)
- moved C5 54.4 mm to (-0.35, 6.85)
- moved R3 54.4 mm to (-11.1, 6.93)
- moved R4 54.4 mm to (-14.7, 7.03)
- moved R5 54.4 mm to (-7.41, 7.03)
- moved R7 54.4 mm to (-4.41, 7.03)
- moved U2 54.4 mm to (-17.1, 10.9)
- moved L36 48.2 mm to (-12.9, 63.6)
- moved RED1 45.0 mm to (152.7, 13.1)
- moved D29 43.2 mm to (142.7, 13.1)
- moved D26 42.8 mm to (132.7, 13.1)
- moved U1 15.6 mm to (144.1, 54.2)
- moved J1 12.5 mm to (29.9, 16.4)
- moved C1 10.5 mm to (110.4, 0.21)
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Connections:
- U1 pad 32: Net-(R10-Pad1) -> Net-(BZ1-Pad1)
Other:
- board size 159.6 x 117 mm -> 159.6 x 120.9 mm

Commit message: schematic final_4
Parts:
- removed the L2 at (52.1, -27.9)
- removed the L5 at (19.4, 22.9)
- removed the L7 at (47.4, 22.8)
- removed the L7 at (33.2, 23.1)
- removed the REF** at (149.6, -8.15)
- added L37: WS2812_LED, keebio_parts:WS2812B, F.Cu at (59.5, 12.1)
- added L38: WS2812_LED, keebio_parts:WS2812B, F.Cu at (46.0, 14.5)
- added L39: WS2812_LED, keebio_parts:WS2812B, F.Cu at (33.8, 16.2)
- added L40: WS2812_LED, keebio_parts:WS2812B, F.Cu at (84.0, 11.0)
- added L41: WS2812_LED, keebio_parts:WS2812B, F.Cu at (97.5, 14.0)
- added L42: WS2812_LED, keebio_parts:WS2812B, F.Cu at (109.8, 15.5)
- added L43: WS2812_LED, keebio_parts:WS2812B, F.Cu at (122.0, 17.5)
- BZ1: footprint Buzzer_Beeper:MagneticBuzzer_PUI_AT-0927-TT-6-R -> reversible-kicad-footprints:Piezo-KLJ-1625
- L32: value SK6812_mini -> WS2812_LED; footprint keebio_parts:SK6812-MINI-E -> keebio_parts:WS2812B
- L36: moved to F.Cu
- moved BZ1 75.7 mm to (66.1, 80.0), turned to 90 degrees
- moved L32 66.5 mm to (71.8, 11.0), turned to 180 degrees
- moved RESET_SW1 62.2 mm to (208.4, 68.7)
- moved RESET_SW1 62.2 mm to (226.3, 66.6)
- moved L36 57.0 mm to (21.5, 18.2)
- moved D28 51.4 mm to (81.6, -17.8)
- moved L4 17.9 mm to (-27.7, 41.2)
- moved D26 10.4 mm to (132.7, 23.5)
- moved D29 10.4 mm to (142.7, 23.5)
- moved RED1 10.4 mm to (152.7, 23.5)
- moved J3 9.47 mm to (143.7, 39.8)
- moved U1 9.47 mm to (143.8, 63.7)
- moved J1 8.28 mm to (38.1, 17.8)
- moved SW19 1.84 mm to (61.8, 95.0)
Connections:
- L32 pad 2: GND -> Net-(L32-Pad2)
- L32 pad 3: Net-(L31-Pad1) -> Net-(L32-Pad3)
Other:
- board size 159.6 x 120.9 mm -> 159.6 x 123.3 mm
- board text added: "monarch rev1.0"
- board text removed: "endless v1.0"

Commit message: monarch update
Parts:
- removed D28: Blue, LED_THT:LED_D3.0mm
- removed D29: Yellow, LED_THT:LED_D3.0mm
- removed the RESET_SW1 at (226.3, 66.6)
- added Boot1: SW_PUSH, Button_Switch_SMD:SW_Push_1P1T_NO_6x6mm_H9.5mm, F.Cu at (134.4, 57.1)
- added D27: Yellow, LED_THT:LED_D3.0mm, F.Cu at (142.6, 23.4)
- added H10: Hole, MountingHole:MountingHole_2.2mm_M2, F.Cu at (73.5, 92.5)
- added H7: Hole, MountingHole:MountingHole_2.2mm_M2, F.Cu at (109.5, 43.2)
- added H8: Hole, MountingHole:MountingHole_2.2mm_M2, F.Cu at (108.9, 82.0)
- added H9: Hole, MountingHole:MountingHole_2.2mm_M2, F.Cu at (165.0, 126.7)
- BZ1: footprint reversible-kicad-footprints:Piezo-KLJ-1625 -> private:Buzzer
- moved L5 180.5 mm to (157.5, 124.9)
- moved C7 178.2 mm to (30.0, 30.0)
- moved L6 175.2 mm to (167.5, 103.3)
- moved L33 174.5 mm to (155.2, 43.2)
- moved C8 169.5 mm to (39.0, 25.0)
- moved C5 166.3 mm to (148.1, 81.8)
- moved L4 166.0 mm to (119.5, 117.9)
- moved L8 164.8 mm to (155.4, 63.3)
- moved R4 160.5 mm to (131.4, 73.2), turned to 180 degrees
- moved D25 157.9 mm to (20.8, 30.0)
- moved R3 155.6 mm to (131.4, 69.5), turned to 180 degrees
- moved L34 155.5 mm to (155.2, 28.3)
- moved L7 155.2 mm to (155.1, 80.1)
- moved F1 154.6 mm to (30.0, 25.0)
- moved L35 153.3 mm to (138.7, 19.1)
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- renumbered H2 to H9
Connections:
- R6 pad 2: Net-(D29-Pad1) -> Net-(D27-Pad1)
- U1 pad 27: Net-(R9-Pad1) -> Net-(R6-Pad1)
- U1 pad 8: Net-(R6-Pad1) -> Net-(Boot1-Pad1)
