File: deskdocker_v1.sch (KiCad schematic (older format))
At the start: 121 parts, among them J1 USB_C_Receptacle_USB2.0, J2 USB_C_Receptacle_USB2.0, J3 OLED, SW1 SW_PUSH, SW10 SW_PUSH, SW11 SW_PUSH, SW12 SW_PUSH, SW13 SW_PUSH, SW14 SW_PUSH, SW15 SW_PUSH, SW16 SW_PUSH, SW17 SW_PUSH, SW18 SW_PUSH, SW19 SW_PUSH, SW2 SW_PUSH, SW20 SW_PUSH, SW21 SW_PUSH, SW22 SW_PUSH, SW23 SW_PUSH, SW24 SW_PUSH, SW25 Rotary_Encoder_Switch, SW3 SW_PUSH, SW4 SW_PUSH, SW5 SW_PUSH, SW6 SW_PUSH, SW7 SW_PUSH, SW8 SW_PUSH, SW9 SW_PUSH, U1 ATMEGA32U4, U2 MIC5219-5.0YMM, X1 16Mhz

Commit message: init commit
Parts:
- removed JP2, JP3, JP4, JP5, JP6, JP7, JP8, JP9: Jumper_NO_Small, symbol Device:Jumper_NO_Small
- added D26, D29: Green, symbol Device:LED
- added D27, D28: LED, symbol Device:LED
- added R6, R8: 330, Resistor_SMD:R_0805_2012Metric, symbol Device:R_Small_US
- J1, J2: footprint Connector_USB:USB_C_Receptacle_GCT_USB4085 -> Connector_USB:USB_C_Receptacle_HRO_TYPE-C-31-M-12
- J3: footprint (none) -> Display:Generic_0.96in-128x64-OLED-Display-IIC
Connections:
- net +3V3 is gone; now on net VCC: R2.1
- net ROW0 is gone; now on net A3: D1.1 (K), D2.1 (K), D3.1 (K), D4.1 (K), D5.1 (K), D6.1 (K)
- net ROW1 is gone; now on net A2: D10.1 (K), D11.1 (K), D12.1 (K), D7.1 (K), D8.1 (K), D9.1 (K)
- net ROW2 is gone; now on net A1: D13.1 (K), D14.1 (K), D15.1 (K), D16.1 (K), D17.1 (K), D18.1 (K)
- net ROW3 is gone; now on net A0: D19.1 (K), D20.1 (K), D21.1 (K), D22.1 (K), D23.1 (K), D24.1 (K)
- net +5V: no longer C1.1, C19.2, C3.2, C5.2, RESET_SW1.2, U1.23 (GND), U1.33 (~HWB/PE2), U1.35 (GND), U1.43 (GND), U1.5 (UGnd)
- net SCL: now also J3.3
- net SDA: now also J3.4
- net VCC: now also J3.2, D26.2 (A), D29.2 (A)
- net at U1.22 (PD5/XCK1): now also R8.1
- net at U1.8 (PB0/SS): now also R6.1
- net GND: now reaches J3.1
- net GND: now also C1.1, C19.2, C3.2, C5.2, RESET_SW1.2, U1.23 (GND), U1.33 (~HWB/PE2), U1.35 (GND), U1.43 (GND), U1.5 (UGnd)
- new net: D26.1 (K), R8.2
- new net: D29.1 (K), R6.2
Other:
- moved on the sheet: C1, C2, C4, C5, R2, X1

Commit message: schematic done -ish?
Connections:
- net +5V: no longer C2.2, C4.2, C6.2, C7.2, C8.2, J1.A1 (GND), J1.A12 (GND), J1.B1 (GND), J1.B12 (GND), J1.S1 (SHIELD), L1.2 (GND), L15.2 (GND), L16.2 (GND), L17.2 (GND), L18.2 (GND), L19.2 (GND), L2.2 (GND), L20.2 (GND), L21.2 (GND), L22.2 (GND), L23.2 (GND), L24.2 (GND), L25.2 (GND), L26.2 (GND), L27.2 (GND), L28.2 (GND), L29.2 (GND), L3.2 (GND), L30.2 (GND), L31.2 (GND), L32.2 (GND), L4.2 (GND), L5.2 (GND), L6.2 (GND), L7.2 (GND), L8.2 (GND), RED1.1 (K), U1.15 (GND), U2.5 (GND), U2.6 (GND), U2.7 (GND), U2.8 (GND)
- net GND: now also C2.2, C4.2, C6.2, C7.2, C8.2, J1.A1 (GND), J1.A12 (GND), J1.B1 (GND), J1.B12 (GND), J1.S1 (SHIELD), L1.2 (GND), L15.2 (GND), L16.2 (GND), L17.2 (GND), L18.2 (GND), L19.2 (GND), L2.2 (GND), L20.2 (GND), L21.2 (GND), L22.2 (GND), L23.2 (GND), L24.2 (GND), L25.2 (GND), L26.2 (GND), L27.2 (GND), L28.2 (GND), L29.2 (GND), L3.2 (GND), L30.2 (GND), L31.2 (GND), L32.2 (GND), L4.2 (GND), L5.2 (GND), L6.2 (GND), L7.2 (GND), L8.2 (GND), RED1.1 (K), U1.15 (GND), U2.5 (GND), U2.6 (GND), U2.7 (GND), U2.8 (GND)
Changed lines of the file:
@@
 	1500 5850 1500 6600
 Connection ~ 1500 5850
-$Comp
-L keyboard_parts:GND #PWR0103
-U 1 1 6057E641
-P 11050 650
-F 0 "#PWR0103" H 11050 700 20  0001 C CNN
-F 1 "GND" H 11050 709 30  0000 C CNN
-F 2 "" H 11050 650 60  0000 C CNN
-F 3 "" H 11050 650 60  0000 C CNN
-	1    11050 650
-	-1   0    0    1
-$EndComp
 Text GLabel 4350 4750 1    50   Input ~ 0
 COL4
@@
 	1    0    0    -1
 $EndComp
-Connection ~ 10700 650
-Wire Wire Line
-	10700 650  11050 650
 Wire Wire Line
 	9400 650  10700 650
@@
 Wire Wire Line
 	7450 2200 7450 2450
-$Comp
-L keyboard_parts:GND #PWR0112
-U 1 1 60652038
-P 5750 2450
-F 0 "#PWR0112" H 5750 2500 20  0001 C CNN
-F 1 "GND" H 5750 2509 30  0000 C CNN
-F 2 "" H 5750 2450 60  0000 C CNN
-F 3 "" H 5750 2450 60  0000 C CNN
-	1    5750 2450
-	1    0    0    -1
-$EndComp
 Connection ~ 10100 1500
 Wire Wire Line
@@
 Wire Wire Line
 	9900 4100 9900 4250
-$Comp
-L keyboard_parts:GND #PWR04
-U 1 1 60898964
-P 10700 3750
-F 0 "#PWR04" H 10700 3800 20  0001 C CNN
-F 1 "GND" H 10700 3809 30  0000 C CNN
-F 2 "" H 10700 3750 60  0000 C CNN
-F 3 "" H 10700 3750 60  0000 C CNN
-	1    10700 3750
-	-1   0    0    1
-$EndComp
 Wire Wire Line
 	10700 3750 10400 3750
@@
 Wire Wire Line
 	9100 4750 9900 4750
-$Comp
-L keyboard_parts:GND #PWR05
-U 1 1 609D54AC
-P 10700 4750
-F 0 "#PWR05" H 10700 4800 20  0001 C CNN
-F 1 "GND" H 10700 4809 30  0000 C CNN
-F 2 "" H 10700 4750 60  0000 C CNN
-F 3 "" H 10700 4750 60  0000 C CNN
-	1    10700 4750
-	-1   0    0    1
-$EndComp
 Wire Wire Line
 	9900 4750 10700 4750
@@
 Wire Wire Line
 	9600 2650 8800 2650
-$Comp
-L keyboard_parts:GND #PWR0101
-U 1 1 605EDDF6
-P -3400 4050
-F 0 "#PWR0101" H -3400 4100 20  0001 C CNN
-F 1 "GND" H -3400 3950 30  0000 C CNN
-F 2 "" H -3400 4050 60  0000 C CNN
-F 3 "" H -3400 4050 60  0000 C CNN
-	1    -3400 4050
-	1    0    0    -1
-$EndComp
 Wire Wire Line
 	-1000 2000 -900 2000
@@
 Text GLabel -3550 1200 0    50   Input ~ 0
 D-
-$Comp
-L keyboard_parts:GND #PWR0106
-U 1 1 608BE9BC
-P -5850 2550
-F 0 "#PWR0106" H -5850 2600 20  0001 C CNN
-F 1 "GND" V -5850 2350 30  0000 L CNN
-F 2 "" H -5850 2550 60  0000 C CNN
-F 3 "" H -5850 2550 60  0000 C CNN
-	1    -5850 2550
-	0    1    1    0
-$EndComp
 Text GLabel 3850 1300 2    50   Input ~ 0
 D-
@@
 	1    0    0    -1
 $EndComp
-$Comp
-L keyboard_parts:GND #PWR0110
-U 1 1 606E47AB
-P 2200 2250
-F 0 "#PWR0110" H 2200 2300 20  0001 C CNN
-F 1 "GND" H 2300 2250 30  0000 C CNN
-F 2 "" H 2200 2250 60  0000 C CNN
-F 3 "" H 2200 2250 60  0000 C CNN
-	1    2200 2250
-	1    0    0    -1
-$EndComp
-$Comp
-L keyboard_parts:GND #PWR0111
-U 1 1 6070C745
-P 2500 2250
-F 0 "#PWR0111" H 2500 2300 20  0001 C CNN
-F 1 "GND" H 2600 2250 30  0000 C CNN
-F 2 "" H 2500 2250 60  0000 C CNN
-F 3 "" H 2500 2250 60  0000 C CNN
-	1    2500 2250
-	1    0    0    -1
-$EndComp
 Wire Wire Line
 	3100 1250 3150 1250
@@
 	-2300 -550 -2000 -550
 Connection ~ -2300 -550
-$Comp
-L keyboard_parts:GND #PWR0116
-U 1 1 60897F06
-P -1600 -50
-F 0 "#PWR0116" H -1600 0   20  0001 C CNN
-F 1 "GND" H -1600 -150 30  0000 C CNN
-F 2 "" H -1600 -50 60  0000 C CNN
-F 3 "" H -1600 -50 60  0000 C CNN
-	1    -1600 -50
-	1    0    0    -1
-$EndComp
 Wire Wire Line
 	-1600 -50  -1600 -150
@@
 	1    0    0    -1
 $EndComp
-$Comp
-L keyboard_parts:GND #PWR0118
-U 1 1 609E6F55
-P -950 -50
-F 0 "#PWR0118" H -950 0   20  0001 C CNN
-F 1 "GND" H -950 -150 30  0000 C CNN
-F 2 "" H -950 -50 60  0000 C CNN
-F 3 "" H -950 -50 60  0000 C CNN
-	1    -950 -50
-	1    0    0    -1
-$EndComp
 Wire Wire Line
 	-1300 -550 -950 -550
@@
 	0    -550 0    -450
 Connection ~ -450 -550
-$Comp
-L keyboard_parts:GND #PWR0119
-U 1 1 60AEAAFC
-P -450 -50
-F 0 "#PWR0119" H -450 0   20  0001 C CNN
-F 1 "GND" H -450 -150 30  0000 C CNN
-F 2 "" H -450 -50 60  0000 C CNN
-F 3 "" H -450 -50 60  0000 C CNN
-	1    -450 -50
-	1    0    0    -1
-$EndComp
 Wire Wire Line
 	-450 -150 -450 -50
-$Comp
-L keyboard_parts:GND #PWR0120
-U 1 1 60B6DE10
-P 0 -50
-F 0 "#PWR0120" H 0   0   20  0001 C CNN
-F 1 "GND" H 0   -150 30  0000 C CNN
-F 2 "" H 0   -50 60  0000 C CNN
-F 3 "" H 0   -50 60  0000 C CNN
-	1    0    -50
-	1    0    0    -1
-$EndComp
 Wire Wire Line
 	0    -150 0    -50
@@
 	1    600  200
 	0    -1   -1   0
-$EndComp
-$Comp
-L keyboard_parts:GND #PWR0122
-U 1 1 60BCCF66
-P 600 450
-F 0 "#PWR0122" H 600 500 20  0001 C CNN
-F 1 "GND" H 600 350 30  0000 C CNN
-F 2 "" H 600 450 60  0000 C CNN
-F 3 "" H 600 450 60  0000 C CNN
-	1    600  450
-	1    0    0    -1
 $EndComp
 Wire Wire Line
@@
 $EndComp
 $Comp
-L power:GND #PWR?
+L power:GND #PWR0104
 U 1 1 608216F9
 P -4200 600
-F 0 "#PWR?" H -4200 350 50  0001 C CNN
+F 0 "#PWR0104" H -4200 350 50  0001 C CNN
 F 1 "GND" H -4195 427 50  0000 C CNN
 F 2 "" H -4200 600 50  0001 C CNN
@@
 $EndComp
 $Comp
-L power:GND #PWR?
+L power:GND #PWR0105
 U 1 1 608914A8
 P -3900 600
-F 0 "#PWR?" H -3900 350 50  0001 C CNN
+F 0 "#PWR0105" H -3900 350 50  0001 C CNN
 F 1 "GND" H -3895 427 50  0000 C CNN
 F 2 "" H -3900 600 50  0001 C CNN
@@
 $EndComp
 $Comp
-L power:GND #PWR?
+L power:GND #PWR0107
 U 1 1 60901457
 P -650 600
-F 0 "#PWR?" H -650 350 50  0001 C CNN
+F 0 "#PWR0107" H -650 350 50  0001 C CNN
 F 1 "GND" H -645 427 50  0000 C CNN
 F 2 "" H -650 600 50  0001 C CNN
@@
 $EndComp
 $Comp
-L power:GND #PWR?
+L power:GND #PWR0110
 U 1 1 6097058F
 P -400 600
-F 0 "#PWR?" H -400 350 50  0001 C CNN
+F 0 "#PWR0110" H -400 350 50  0001 C CNN
 F 1 "GND" H -395 427 50  0000 C CNN
 F 2 "" H -400 600 50  0001 C CNN
@@
 $EndComp
 $Comp
-L power:GND #PWR?
+L power:GND #PWR0111
 U 1 1 609E183F
 P 1950 2700
-F 0 "#PWR?" H 1950 2450 50  0001 C CNN
+F 0 "#PWR0111" H 1950 2450 50  0001 C CNN
 F 1 "GND" H 1955 2527 50  0000 C CNN
 F 2 "" H 1950 2700 50  0001 C CNN
@@
 $EndComp
 $Comp
-L power:GND #PWR?
+L power:GND #PWR0114
 U 1 1 60A517B4
 P 1850 3750
-F 0 "#PWR?" H 1850 3500 50  0001 C CNN
+F 0 "#PWR0114" H 1850 3500 50  0001 C CNN
 F 1 "GND" V 1850 3550 50  0000 C CNN
 F 2 "" H 1850 3750 50  0001 C CNN
@@
 	0    -1   -1   0
 $EndComp
+$Comp
+L power:GND #PWR0125
+U 1 1 60ACEA75
+P 2200 2250
+F 0 "#PWR0125" H 2200 2000 50  0001 C CNN
+F 1 "GND" H 2205 2077 50  0000 C CNN
+F 2 "" H 2200 2250 50  0001 C CNN
+F 3 "" H 2200 2250 50  0001 C CNN
+	1    2200 2250
+	1    0    0    -1
+$EndComp
+$Comp
+L power:GND #PWR0128
+U 1 1 60B0610C
+P 2500 2250
+F 0 "#PWR0128" H 2500 2000 50  0001 C CNN
+F 1 "GND" H 2505 2077 50  0000 C CNN
+F 2 "" H 2500 2250 50  0001 C CNN
+F 3 "" H 2500 2250 50  0001 C CNN
+	1    2500 2250
+	1    0    0    -1
+$EndComp
+Connection ~ 10700 650
+Wire Wire Line
+	10700 650  11050 650
+$Comp
+L power:GND #PWR?
+U 1 1 60B7B7D5
+P 11050 650
+F 0 "#PWR?" H 11050 400 50  0001 C CNN
+F 1 "GND" H 11055 477 50  0000 C CNN
+F 2 "" H 11050 650 50  0001 C CNN
+F 3 "" H 11050 650 50  0001 C CNN
+	1    11050 650
+	-1   0    0    1
+$EndComp
+$Comp
+L power:GND #PWR?
+U 1 1 60BB3973
+P 10700 3750
+F 0 "#PWR?" H 10700 3500 50  0001 C CNN
+F 1 "GND" H 10705 3577 50  0000 C CNN
+F 2 "" H 10700 3750 50  0001 C CNN
+F 3 "" H 10700 3750 50  0001 C CNN
+	1    10700 3750
+	-1   0    0    1
+$EndComp
+$Comp
+L power:GND #PWR?
+U 1 1 60BEB6B1
+P 10700 4750
+F 0 "#PWR?" H 10700 4500 50  0001 C CNN
+F 1 "GND" H 10705 4577 50  0000 C CNN
+F 2 "" H 10700 4750 50  0001 C CNN
+F 3 "" H 10700 4750 50  0001 C CNN
+	1    10700 4750
+	-1   0    0    1
+$EndComp
+$Comp
+L power:GND #PWR?
+U 1 1 60C24D30
+P 5750 2450
+F 0 "#PWR?" H 5750 2200 50  0001 C CNN
+F 1 "GND" H 5755 2277 50  0000 C CNN
+F 2 "" H 5750 2450 50  0001 C CNN
+F 3 "" H 5750 2450 50  0001 C CNN
+	1    5750 2450
+	-1   0    0    1
+$EndComp
+$Comp
+L power:GND #PWR?
+U 1 1 60CD4DDF
+P -3400 4050
+F 0 "#PWR?" H -3400 3800 50  0001 C CNN
+F 1 "GND" H -3395 3877 50  0000 C CNN
+F 2 "" H -3400 4050 50  0001 C CNN
+F 3 "" H -3400 4050 50  0001 C CNN
+	1    -3400 4050
+	1    0    0    -1
+$EndComp
+$Comp
+L power:GND #PWR?
+U 1 1 60D45238
+P -1600 -50
+F 0 "#PWR?" H -1600 -300 50  0001 C CNN
+F 1 "GND" H -1595 -223 50  0000 C CNN
+F 2 "" H -1600 -50 50  0001 C CNN
+F 3 "" H -1600 -50 50  0001 C CNN
+	1    -1600 -50
+	1    0    0    -1
+$EndComp
+$Comp
+L power:GND #PWR?
+U 1 1 60D7C583
+P -950 -50
+F 0 "#PWR?" H -950 -300 50  0001 C CNN
+F 1 "GND" H -945 -223 50  0000 C CNN
+F 2 "" H -950 -50 50  0001 C CNN
+F 3 "" H -950 -50 50  0001 C CNN
+	1    -950 -50
+	1    0    0    -1
+$EndComp
+$Comp
+L power:GND #PWR?
+U 1 1 60DB3EA6
+P -450 -50
+F 0 "#PWR?" H -450 -300 50  0001 C CNN
+F 1 "GND" H -445 -223 50  0000 C CNN
+F 2 "" H -450 -50 50  0001 C CNN
+F 3 "" H -450 -50 50  0001 C CNN
+	1    -450 -50
+	1    0    0    -1
+$EndComp
+$Comp
+L power:GND #PWR?
+U 1 1 60DEB135
+P 0 -50
+F 0 "#PWR?" H 0   -300 50  0001 C CNN
+F 1 "GND" H 5   -223 50  0000 C CNN
+F 2 "" H 0   -50 50  0001 C CNN
+F 3 "" H 0   -50 50  0001 C CNN
+	1    0    -50
+	1    0    0    -1
+$EndComp
+$Comp
+L power:GND #PWR?
+U 1 1 60E22BFC
+P 600 450
+F 0 "#PWR?" H 600 200 50  0001 C CNN
+F 1 "GND" H 605 277 50  0000 C CNN
+F 2 "" H 600 450 50  0001 C CNN
+F 3 "" H 600 450 50  0001 C CNN
+	1    600  450
+	1    0    0    -1
+$EndComp
+$Comp
+L power:GND #PWR?
+U 1 1 60E5C8DE
+P -5850 2550
+F 0 "#PWR?" H -5850 2300 50  0001 C CNN
+F 1 "GND" H -5845 2377 50  0000 C CNN
+F 2 "" H -5850 2550 50  0001 C CNN
+F 3 "" H -5850 2550 50  0001 C CNN
+	1    -5850 2550
+	0    1    1    0
+$EndComp
 $EndSCHEMATC

Commit message: schematic pre-final
Parts:
- removed SW19: SW_PUSH, keyswitches:Kailh_socket_MX, symbol keyboard_parts:SW_PUSH
- added R10, R9: 330, Resistor_SMD:R_0805_2012Metric, symbol Device:R_Small_US
- added R11, R12: 5.1k, Resistor_SMD:R_0805_2012Metric, symbol Device:R_US
- D27: value LED -> Orange
- D28: value LED -> Blue
- D29: value Green -> Yellow
- renumbered SW25 to SW19
Connections:
- net D4 is gone; now on net COL0: U1.25 (ICP1/PD4)
- net D5 is gone; now on net COL1: U1.31 (PC6)
- net D7 is gone; now on net COL3: U1.1 (PE6/AIN0)
- net D8 is gone; now on net COL4: U1.28 (PB4)
- net LED is gone; now on net D9: L1.3 (DIN)
- net SCL is gone; now on net D3: J3.3
- net SDA is gone; now on net D2: J3.4
- net +5V: now also R11.1, R12.1
- net COL0: now also SW19.S2
- net COL2: now also U1.26 (T1/PD6)
- net D10: now also L9.3 (DIN)
- net GND: now also J2.A1 (GND), J2.A12 (GND), J2.B1 (GND), J2.B12 (GND), J2.S1 (SHIELD), SW19.C
- net RX: now also J2.A6 (D+), J2.B7 (D-)
- net VCC: now also D27.2 (A), D28.2 (A), J2.A4 (VBUS), J2.A9 (VBUS), J2.B4 (VBUS), J2.B9 (VBUS)
- net at L8.1 (DOUT): no longer L9.3 (DIN)
- net at U1.32 (PC7): now also R10.1
- net A4: now reaches U1.40 (PF1)
- net A4: now also SW19.A
- net A5: now reaches U1.41 (PF0)
- net A5: now also SW19.B
- net at J2.A5 (CC1): now also R11.2
- net at J2.B5 (CC2): now also R12.2
- net at D27.1 (K): now also R10.2
- net at D28.1 (K): now also R9.2
- net at D19.2 (A): now also SW19.S1
- net D6: no longer names the net of U1.27 (T0/PD7)
- net D6: now also R9.1
- no-connect marks 7 -> 8
Other:
- note removed: "A4"
- note removed: "A5"
- note removed: "D12"
- note removed: "D13"
- moved on the sheet: C1, C19, C2, C3, C4, C5, C6, C7, C8, D19, D25, D26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

Commit message: schematic final_1
Parts:
- removed R11, R12: 5.1k, Resistor_SMD:R_0805_2012Metric, symbol Device:R_US
- added L33, L34, L35, L36: WS2812_LED, keebio_parts:WS2812B, symbol keyboard_parts:WS2812_LED
- D26, D27, D28, D29: footprint (none) -> LED_SMD:LED_0603_1608Metric
- SW23, SW24: footprint keebio_parts:MX-Alps_Switch_Cutout-1u_2u -> keyswitches:Kailh_socket_MX
Connections:
- net +5V: now also J2.A5 (CC1), J2.B5 (CC2)
- net GND: now also L33.2 (GND), L34.2 (GND), L35.2 (GND), L36.2 (GND)
- net VCC: now also L33.4 (VCC), L34.4 (VCC), L35.4 (VCC), L36.4 (VCC)
- net at L8.1 (DOUT): now also L33.3 (DIN)
- new net: L33.1 (DOUT), L34.3 (DIN)
- new net: L34.1 (DOUT), L35.3 (DIN)
- new net: L35.1 (DOUT), L36.3 (DIN)
- no-connect marks 8 -> 10
Other:
- moved on the sheet: L1, L10, L11, L12, L13, L14, L15, L16, L17, L18, L19, L2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

Commit message: schematic final_3
Parts:
- removed D27: Orange, LED_SMD:LED_0603_1608Metric, symbol Device:LED
- removed H1, H2, H3, H4, H5, H6: Hole, MountingHole:MountingHole_2.2mm_M2, symbol keebio:Hole
- removed R10: 330, Resistor_SMD:R_0805_2012Metric, symbol Device:R_Small_US
- added BZ1: Buzzer, Buzzer_Beeper:MagneticBuzzer_PUI_AT-0927-TT-6-R, symbol Device:Buzzer
- D26, D28, D29, RED1: footprint LED_SMD:LED_0603_1608Metric -> LED_THT:LED_D3.0mm
- J1, J2: footprint Connector_USB:USB_C_Receptacle_HRO_TYPE-C-31-M-12 -> private:USB_C_TH_6pin
- RESET_SW1: footprint keebio_parts:SW_Tactile_SPST_Angled_MJTP1117 -> Button_Switch_SMD:SW_Push_1P1T_NO_6x6mm_H9.5mm
- SW19: value Rotary_Encoder_Switch -> Rotary_Encoder
Connections:
- net GND: now also BZ1.2 (+)
- net at U1.32 (PC7): now also BZ1.1 (-)
Other:
- moved on the sheet: C1, C19, C2, C3, C4, C5, C6, C7, C8, D25, D26, D28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

Commit message: schematic final_4
Parts:
- removed L32: SK6812_mini, keebio_parts:SK6812-MINI-E, symbol keyboard_parts:SK6812_mini
- added L32, L37, L38, L39, L40, L41, L42, L43: WS2812_LED, keebio_parts:WS2812B, symbol keyboard_parts:WS2812_LED
- BZ1: footprint Buzzer_Beeper:MagneticBuzzer_PUI_AT-0927-TT-6-R -> reversible-kicad-footprints:Piezo-KLJ-1625
Connections:
- net VCC: now also L32.4 (VCC), L37.4 (VCC), L38.4 (VCC), L39.4 (VCC), L40.4 (VCC), L41.4 (VCC), L42.4 (VCC), L43.4 (VCC)
- net at L36.1 (DOUT): now also L39.3 (DIN)
- new net: L38.3 (DIN), L39.1 (DOUT)
- new net: L32.2 (GND), L37.2 (GND), L38.2 (GND), L39.2 (GND), L40.2 (GND), L41.2 (GND), L42.2 (GND), L43.2 (GND)
- new net: L37.3 (DIN), L38.1 (DOUT)
- new net: L32.3 (DIN), L37.1 (DOUT)
- new net: L32.1 (DOUT), L40.3 (DIN)
- new net: L40.1 (DOUT), L41.3 (DIN)
- new net: L41.1 (DOUT), L42.3 (DIN)
- new net: L42.1 (DOUT), L43.3 (DIN)
Other:
- moved on the sheet: L1, L2, L3, L33, L34, L35, L36, L4, L5, L6, L7, L8

Commit message: monarch update
Parts:
- removed D28: Blue, LED_THT:LED_D3.0mm, symbol Device:LED
- removed D29: Yellow, LED_THT:LED_D3.0mm, symbol Device:LED
- removed R9: 330, Resistor_SMD:R_0805_2012Metric, symbol Device:R_Small_US
- added Boot1: SW_PUSH, Button_Switch_SMD:SW_Push_1P1T_NO_6x6mm_H9.5mm, symbol keyboard_parts:SW_PUSH
- added D27: Yellow, LED_THT:LED_D3.0mm, symbol Device:LED
- BZ1: footprint reversible-kicad-footprints:Piezo-KLJ-1625 -> private:Buzzer
Connections:
- net GND: now also Boot1.2
- net VCC: now also D27.2 (A)
- net at U1.27 (T0/PD7): now also R6.1
- net at U1.8 (PB0/SS): now also Boot1.1; no longer R6.1
- net at R6.2: now also D27.1 (K)
Changed lines of the file:
@@
 	1    0    0    -1
 $EndComp
-$Comp
-L power:VCC #PWR0115
-U 1 1 608EE946
-P -4900 1100
-F 0 "#PWR0115" H -4900 950 50  0001 C CNN
-F 1 "VCC" H -4885 1273 50  0000 C CNN
-F 2 "" H -4900 1100 50  0001 C CNN
-F 3 "" H -4900 1100 50  0001 C CNN
-	1    -4900 1100
-	1    0    0    -1
-$EndComp
-Wire Wire Line
-	-4900 1700 -4900 1600
-$Comp
-L Device:R_Small_US R6
-U 1 1 608EE94D
-P -4900 1800
-F 0 "R6" H -4832 1846 50  0000 L CNN
-F 1 "330" H -4832 1755 50  0000 L CNN
-F 2 "Resistor_SMD:R_0805_2012Metric" H -4900 1800 50  0001 C CNN
-F 3 "~" H -4900 1800 50  0001 C CNN
-	1    -4900 1800
-	-1   0    0    1
-$EndComp
-Wire Wire Line
-	-4900 1300 -4900 1100
-$Comp
-L Device:LED D29
-U 1 1 608EE955
-P -4900 1450
-F 0 "D29" V -4953 1530 50  0000 L CNN
-F 1 "Yellow" V -4862 1530 50  0000 L CNN
-F 2 "LED_THT:LED_D3.0mm" H -4900 1450 50  0001 C CNN
-F 3 "~" H -4900 1450 50  0001 C CNN
-	1    -4900 1450
-	0    -1   -1   0
-$EndComp
 Wire Wire Line
 	-4550 2000 -4550 1550
@@
 D+
 Wire Wire Line
-	-4900 2200 -4900 1900
-Wire Wire Line
 	-3750 1100 -3750 2800
 Text GLabel -3900 2300 0    50   Input ~ 0
@@
 Text GLabel -4900 -900 0    50   Input ~ 0
 UVCC
-$Comp
-L keyboard_parts:PPTC F1
-U 1 1 6060CBCC
-P -4250 -900
-F 0 "F1" H -4250 -660 50  0000 C CNN
-F 1 "PPTC" H -4250 -751 50  0000 C CNN
-F 2 "Fuse:Fuse_1206_3216Metric" V -4250 -900 60  0001 C CNN
-F 3 "" V -4250 -900 60  0000 C CNN
-	1    -4250 -900
-	1    0    0    -1
-$EndComp
 Connection ~ -2000 -550
 Connection ~ 4950 7650
@@
 F 0 "BZ1" V 150 3750 50  0000 L CNN
 F 1 "Buzzer" V 50  3700 50  0000 L CNN
-F 2 "reversible-kicad-footprints:Piezo-KLJ-1625" V -125 3950 50  0001 C CNN
+F 2 "private:Buzzer" V -125 3950 50  0001 C CNN
 F 3 "~" V -125 3950 50  0001 C CNN
 	1    -100 3850
@@
 Connection ~ 9550 2000
 Connection ~ 9550 2850
-Wire Wire Line
-	-550 4350 -550 4550
 $Comp
-L power:VCC #PWR0137
-U 1 1 60933AB2
+L keyboard_parts:PPTC F1
+U 1 1 6060CBCC
+P -4250 -900
+F 0 "F1" H -4250 -660 50  0000 C CNN
+F 1 "PPTC" H -4250 -751 50  0000 C CNN
+F 2 "Fuse:Fuse_1206_3216Metric" V -4250 -900 60  0001 C CNN
+F 3 "" V -4250 -900 60  0000 C CNN
+	1    -4250 -900
+	1    0    0    -1
+$EndComp
+$Comp
+L power:VCC #PWR0115
+U 1 1 6084752F
 P -550 4550
-F 0 "#PWR0137" H -550 4400 50  0001 C CNN
+F 0 "#PWR0115" H -550 4400 50  0001 C CNN
 F 1 "VCC" H -535 4723 50  0000 C CNN
 F 2 "" H -550 4550 50  0001 C CNN
@@
 $EndComp
 Wire Wire Line
-	-550 3750 -550 3200
+	-550 3950 -550 4050
+$Comp
+L Device:R_Small_US R6
+U 1 1 60847536
+P -550 3850
+F 0 "R6" H -482 3896 50  0000 L CNN
+F 1 "330" H -482 3805 50  0000 L CNN
+F 2 "Resistor_SMD:R_0805_2012Metric" H -550 3850 50  0001 C CNN
+F 3 "~" H -550 3850 50  0001 C CNN
+	1    -550 3850
+	1    0    0    -1
+$EndComp
+Wire Wire Line
+	-550 4350 -550 4550
 $Comp
-L Device:LED D28
-U 1 1 6065AA39
+L Device:LED D27
+U 1 1 6084753D
 P -550 4200
-F 0 "D28" V -603 4280 50  0000 L CNN
-F 1 "Blue" V -512 4280 50  0000 L CNN
+F 0 "D27" V -603 4280 50  0000 L CNN
+F 1 "Yellow" V -512 4280 50  0000 L CNN
 F 2 "LED_THT:LED_D3.0mm" H -550 4200 50  0001 C CNN
 F 3 "~" H -550 4200 50  0001 C CNN
@@
 $EndComp
 $Comp
-L Device:R_Small_US R9
-U 1 1 607777D2
-P -550 3850
-F 0 "R9" H -482 3896 50  0000 L CNN
-F 1 "330" H -482 3805 50  0000 L CNN
-F 2 "Resistor_SMD:R_0805_2012Metric" H -550 3850 50  0001 C CNN
-F 3 "~" H -550 3850 50  0001 C CNN
-	1    -550 3850
-	1    0    0    -1
+L power:GND #PWR0137
+U 1 1 608DAD16
+P -4900 1100
+F 0 "#PWR0137" H -4900 850 50  0001 C CNN
+F 1 "GND" H -4895 927 50  0000 C CNN
+F 2 "" H -4900 1100 50  0001 C CNN
+F 3 "" H -4900 1100 50  0001 C CNN
+	1    -4900 1100
+	-1   0    0    1
 $EndComp
 Wire Wire Line
-	-550 3950 -550 4050
+	-4900 1300 -4900 1100
+$Comp
+L keyboard_parts:SW_PUSH Boot1
+U 1 1 608DAD1D
+P -4900 1600
+F 0 "Boot1" H -4900 1855 50  0000 C CNN
+F 1 "SW_PUSH" H -4900 1764 50  0000 C CNN
+F 2 "Button_Switch_SMD:SW_Push_1P1T_NO_6x6mm_H9.5mm" H -4900 1600 60  0001 C CNN
+F 3 "" H -4900 1600 60  0000 C CNN
+	1    -4900 1600
+	0    -1   -1   0
+$EndComp
+Wire Wire Line
+	-4900 1900 -4900 2200
+Wire Wire Line
+	-550 3200 -550 3750
 $EndSCHEMATC
