File: monarch.sch (KiCad schematic (older format))
At the start: 123 parts, among them J1 USB_C_Receptacle_USB2.0, J2 USB_C_Receptacle_USB2.0, J3 OLED, SW1 SW_PUSH, SW10 SW_PUSH, SW11 SW_PUSH, SW12 SW_PUSH, SW13 SW_PUSH, SW14 SW_PUSH, SW15 SW_PUSH, SW16 SW_PUSH, SW17 SW_PUSH, SW18 SW_PUSH, SW19 Rotary_Encoder, SW2 SW_PUSH, SW20 SW_PUSH, SW21 SW_PUSH, SW22 SW_PUSH, SW23 SW_PUSH, SW24 SW_PUSH, SW3 SW_PUSH, SW4 SW_PUSH, SW5 SW_PUSH, SW6 SW_PUSH, SW7 SW_PUSH, SW8 SW_PUSH, SW9 SW_PUSH, U1 ATMEGA32U4, U2 MIC5219-5.0YMM, X1 16Mhz

Commit message: pre routing/tracing
Connections:
- wire segments 518 -> 520
Changed lines of the file:
@@
-$EndComp
-$Comp
-L power:GND #PWR0117
-U 1 1 60774B53
-P -4200 -150
-F 0 "#PWR0117" H -4200 -400 50  0001 C CNN
-F 1 "GND" H -4195 -323 50  0000 C CNN
-F 2 "" H -4200 -150 50  0001 C CNN
-F 3 "" H -4200 -150 50  0001 C CNN
-	1    -4200 -150
-	1    0    0    -1
 $EndComp
 $Comp
@@
 $EndComp
 $Comp
-L power:GND #PWR0120
-U 1 1 60C24D30
-P 5200 1150
-F 0 "#PWR0120" H 5200 900 50  0001 C CNN
-F 1 "GND" H 5205 977 50  0000 C CNN
-F 2 "" H 5200 1150 50  0001 C CNN
-F 3 "" H 5200 1150 50  0001 C CNN
-	1    5200 1150
-	-1   0    0    1
-$EndComp
-$Comp
-L power:GND #PWR0122
-U 1 1 60BEB6B1
-P 11450 6200
-F 0 "#PWR0122" H 11450 5950 50  0001 C CNN
-F 1 "GND" H 11455 6027 50  0000 C CNN
-F 2 "" H 11450 6200 50  0001 C CNN
-F 3 "" H 11450 6200 50  0001 C CNN
-	1    11450 6200
-	-1   0    0    1
-$EndComp
-$Comp
-L power:GND #PWR0129
-U 1 1 60BB3973
-P 11450 5200
-F 0 "#PWR0129" H 11450 4950 50  0001 C CNN
-F 1 "GND" H 11455 5027 50  0000 C CNN
-F 2 "" H 11450 5200 50  0001 C CNN
-F 3 "" H 11450 5200 50  0001 C CNN
-	1    11450 5200
-	-1   0    0    1
-$EndComp
-$Comp
-L power:GND #PWR0130
-U 1 1 60B7B7D5
-P 10500 -650
-F 0 "#PWR0130" H 10500 -900 50  0001 C CNN
-F 1 "GND" H 10505 -823 50  0000 C CNN
-F 2 "" H 10500 -650 50  0001 C CNN
-F 3 "" H 10500 -650 50  0001 C CNN
-	1    10500 -650
-	-1   0    0    1
-$EndComp
-Wire Wire Line
-	10150 -650 10500 -650
-Connection ~ 10150 -650
-$Comp
 L power:GND #PWR0128
 U 1 1 60B0610C
@@
 $EndComp
 $Comp
-L power:GND #PWR0110
-U 1 1 6097058F
-P -750 1100
-F 0 "#PWR0110" H -750 850 50  0001 C CNN
-F 1 "GND" H -745 927 50  0000 C CNN
-F 2 "" H -750 1100 50  0001 C CNN
-F 3 "" H -750 1100 50  0001 C CNN
-	1    -750 1100
-	-1   0    0    1
-$EndComp
-$Comp
 L power:GND #PWR0107
 U 1 1 60901457
@@
 	7150 4250 7150 4100
 Wire Wire Line
-	5600 1150 6200 1150
-Wire Wire Line
 	8250 1150 8850 1150
 Wire Wire Line
@@
 Wire Wire Line
 	8250 900  8250 1150
-Wire Wire Line
-	5200 1150 5600 1150
 Wire Wire Line
 	5600 700  5450 700
@@
 Wire Wire Line
 	-550 3200 -550 3750
+Wire Wire Line
+	5200 2850 5600 2850
+Wire Wire Line
+	10550 -650 10150 -650
+$Comp
+L power:GND #PWR0110
+U 1 1 609D5069
+P -750 1100
+F 0 "#PWR0110" H -750 850 50  0001 C CNN
+F 1 "GND" H -745 927 50  0000 C CNN
+F 2 "" H -750 1100 50  0001 C CNN
+F 3 "" H -750 1100 50  0001 C CNN
+	1    -750 1100
+	-1   0    0    1
+$EndComp
+$Comp
+L power:GND #PWR0117
+U 1 1 60A1F198
+P -4200 -150
+F 0 "#PWR0117" H -4200 -400 50  0001 C CNN
+F 1 "GND" H -4195 -323 50  0000 C CNN
+F 2 "" H -4200 -150 50  0001 C CNN
+F 3 "" H -4200 -150 50  0001 C CNN
+	1    -4200 -150
+	1    0    0    -1
+$EndComp
+$Comp
+L power:GND #PWR0130
+U 1 1 60AB47AF
+P 5200 2850
+F 0 "#PWR0130" H 5200 2600 50  0001 C CNN
+F 1 "GND" H 5205 2677 50  0000 C CNN
+F 2 "" H 5200 2850 50  0001 C CNN
+F 3 "" H 5200 2850 50  0001 C CNN
+	1    5200 2850
+	-1   0    0    1
+$EndComp
+Connection ~ 5600 2850
+$Comp
+L power:GND #PWR0140
+U 1 1 60BD4038
+P 10550 -650
+F 0 "#PWR0140" H 10550 -900 50  0001 C CNN
+F 1 "GND" H 10555 -823 50  0000 C CNN
+F 2 "" H 10550 -650 50  0001 C CNN
+F 3 "" H 10550 -650 50  0001 C CNN
+	1    10550 -650
+	-1   0    0    1
+$EndComp
+Wire Wire Line
+	5600 1150 6200 1150
+Wire Wire Line
+	5200 1150 5600 1150
+$Comp
+L power:GND #PWR0120
+U 1 1 60C7A5B9
+P 5200 1150
+F 0 "#PWR0120" H 5200 900 50  0001 C CNN
+F 1 "GND" H 5205 977 50  0000 C CNN
+F 2 "" H 5200 1150 50  0001 C CNN
+F 3 "" H 5200 1150 50  0001 C CNN
+	1    5200 1150
+	-1   0    0    1
+$EndComp
+$Comp
+L power:GND #PWR0122
+U 1 1 608A6779
+P 11450 5200
+F 0 "#PWR0122" H 11450 4950 50  0001 C CNN
+F 1 "GND" H 11455 5027 50  0000 C CNN
+F 2 "" H 11450 5200 50  0001 C CNN
+F 3 "" H 11450 5200 50  0001 C CNN
+	1    11450 5200
+	-1   0    0    1
+$EndComp
+$Comp
+L power:GND #PWR0129
+U 1 1 608ED804
+P 11450 6200
+F 0 "#PWR0129" H 11450 5950 50  0001 C CNN
+F 1 "GND" H 11455 6027 50  0000 C CNN
+F 2 "" H 11450 6200 50  0001 C CNN
+F 3 "" H 11450 6200 50  0001 C CNN
+	1    11450 6200
+	-1   0    0    1
+$EndComp
+$Comp
+L power:GND #PWR?
+U 1 1 6093532B
+P 11400 4100
+F 0 "#PWR?" H 11400 3850 50  0001 C CNN
+F 1 "GND" H 11405 3927 50  0000 C CNN
+F 2 "" H 11400 4100 50  0001 C CNN
+F 3 "" H 11400 4100 50  0001 C CNN
+	1    11400 4100
+	-1   0    0    1
+$EndComp
+Wire Wire Line
+	11400 4100 11150 4100
+Connection ~ 11150 4100
 $EndSCHEMATC

Commit message: start routing
Parts:
- J1, J2: footprint private:USB_C_TH_6pin -> Connector_USB:USB_C_Receptacle_GCT_USB4085
Changed lines of the file:
@@
 Wire Wire Line
 	-6200 3050 -6000 3050
-Connection ~ -5250 3350
-Wire Wire Line
-	-5450 3350 -5250 3350
 Wire Wire Line
 	-6000 3350 -5850 3350
@@
 Wire Wire Line
 	-5850 2750 -6000 2750
-Connection ~ -5250 2750
-Wire Wire Line
-	-5450 2750 -5250 2750
 $Comp
 L keyboard_parts:C C2
@@
 	-5100 3350 -5100 3100
 Wire Wire Line
-	-5250 3350 -5100 3350
-Wire Wire Line
-	-5100 2750 -5250 2750
-Wire Wire Line
 	-5100 3000 -5100 2750
-$Comp
-L keyboard_parts:XTAL X1
-U 1 1 6080F4C1
-P -5250 3050
-F 0 "X1" V -5250 2800 60  0000 L CNN
-F 1 "16Mhz" V -5150 2750 60  0000 L CNN
-F 2 "Crystal:Crystal_SMD_SeikoEpson_FA238-4Pin_3.2x2.5mm" H -5250 3050 60  0001 C CNN
-F 3 "" H -5250 3050 60  0000 C CNN
-	1    -5250 3050
-	0    1    1    0
-$EndComp
-Text GLabel -1000 5700 0    50   Input ~ 0
-A3
 Text GLabel -1000 5850 0    50   Input ~ 0
+A3
+Text GLabel -1000 5700 0    50   Input ~ 0
 A2
 Text GLabel -1000 6000 0    50   Input ~ 0
@@
 F 0 "J1" H 1757 2267 50  0000 C CNN
 F 1 "USB_C_Receptacle_USB2.0" H 1757 2176 50  0000 C CNN
-F 2 "private:USB_C_TH_6pin" H 1800 1400 50  0001 C CNN
+F 2 "Connector_USB:USB_C_Receptacle_GCT_USB4085" H 1800 1400 50  0001 C CNN
 F 3 "https://www.usb.org/sites/default/files/documents/usb_type-c.zip" H 1800 1400 50  0001 C CNN
 	1    1650 1400
@@
 $EndComp
 Wire Wire Line
-	3000 1100 3000 1150
-Connection ~ 3000 1100
-Wire Wire Line
 	2800 1100 3000 1100
 Wire Wire Line
@@
 Wire Wire Line
 	2800 1000 3000 1000
-$Comp
-L keyboard_parts:GND #PWR0124
-U 1 1 606E6309
-P 3000 1150
-F 0 "#PWR0124" H 3000 1200 20  0001 C CNN
-F 1 "GND" H 3100 1150 30  0000 C CNN
-F 2 "" H 3000 1150 60  0000 C CNN
-F 3 "" H 3000 1150 60  0000 C CNN
-	1    3000 1150
-	1    0    0    -1
-$EndComp
 Wire Wire Line
 	2250 1100 2500 1100
@@
 F 0 "J2" H 3957 2267 50  0000 C CNN
 F 1 "USB_C_Receptacle_USB2.0" H 3957 2176 50  0000 C CNN
-F 2 "private:USB_C_TH_6pin" H 4000 1400 50  0001 C CNN
+F 2 "Connector_USB:USB_C_Receptacle_GCT_USB4085" H 4000 1400 50  0001 C CNN
 F 3 "https://www.usb.org/sites/default/files/documents/usb_type-c.zip" H 4000 1400 50  0001 C CNN
 	1    3850 1400
@@
 $EndComp
 $Comp
-L power:GND #PWR?
+L power:GND #PWR0141
 U 1 1 6093532B
 P 11400 4100
-F 0 "#PWR?" H 11400 3850 50  0001 C CNN
+F 0 "#PWR0141" H 11400 3850 50  0001 C CNN
 F 1 "GND" H 11405 3927 50  0000 C CNN
 F 2 "" H 11400 4100 50  0001 C CNN
@@
 	11400 4100 11150 4100
 Connection ~ 11150 4100
+$Comp
+L power:GND #PWR0124
+U 1 1 609A1212
+P 3000 900
+F 0 "#PWR0124" H 3000 650 50  0001 C CNN
+F 1 "GND" H 3005 727 50  0000 C CNN
+F 2 "" H 3000 900 50  0001 C CNN
+F 3 "" H 3000 900 50  0001 C CNN
+	1    3000 900
+	-1   0    0    1
+$EndComp
+Wire Wire Line
+	3000 900  3000 1000
+Connection ~ 3000 1000
+Wire Wire Line
+	-5100 2750 -5250 2750
+Wire Wire Line
+	-5450 2750 -5250 2750
+Connection ~ -5250 2750
+Wire Wire Line
+	-5250 3350 -5100 3350
+Wire Wire Line
+	-5450 3350 -5250 3350
+Connection ~ -5250 3350
+$Comp
+L keyboard_parts:XTAL X1
+U 1 1 6080F4C1
+P -5250 3050
+F 0 "X1" V -5250 2800 60  0000 L CNN
+F 1 "16Mhz" V -5150 2750 60  0000 L CNN
+F 2 "Crystal:Crystal_SMD_SeikoEpson_FA238-4Pin_3.2x2.5mm" H -5250 3050 60  0001 C CNN
+F 3 "" H -5250 3050 60  0000 C CNN
+	1    -5250 3050
+	0    1    1    0
+$EndComp
+Text GLabel -1000 7800 0    50   Input ~ 0
+SCK
+Text GLabel -1000 7950 0    50   Input ~ 0
+TX
 $EndSCHEMATC

Commit message: plate edge case
Connections:
- wire segments 520 -> 521
Changed lines of the file:
@@
 	0    1    1    0
 $EndComp
-Wire Wire Line
-	4650 1100 4650 1150
 Connection ~ 4650 1100
 Wire Wire Line
@@
 Wire Wire Line
 	4450 1000 4650 1000
-$Comp
-L keyboard_parts:GND #PWR0135
-U 1 1 60731FA9
-P 4650 1150
-F 0 "#PWR0135" H 4650 1200 20  0001 C CNN
-F 1 "GND" H 4750 1150 30  0000 C CNN
-F 2 "" H 4650 1150 60  0000 C CNN
-F 3 "" H 4650 1150 60  0000 C CNN
-	1    4650 1150
-	1    0    0    -1
-$EndComp
 NoConn ~ 2250 1900
 NoConn ~ 2250 2000
@@
 Text GLabel -1000 7950 0    50   Input ~ 0
 TX
+$Comp
+L power:GND #PWR?
+U 1 1 6082B89B
+P 4850 1000
+F 0 "#PWR?" H 4850 750 50  0001 C CNN
+F 1 "GND" H 4855 827 50  0000 C CNN
+F 2 "" H 4850 1000 50  0001 C CNN
+F 3 "" H 4850 1000 50  0001 C CNN
+	1    4850 1000
+	-1   0    0    1
+$EndComp
+Wire Wire Line
+	4650 1100 4850 1100
+Wire Wire Line
+	4850 1100 4850 1000
 $EndSCHEMATC

Commit message: rerouting v2
Parts:
- X1: footprint Crystal:Crystal_SMD_SeikoEpson_FA238-4Pin_3.2x2.5mm -> Crystal:Crystal_SMD_7050-4Pin_7.0x5.0mm
Changed lines of the file:
@@
 F 0 "X1" V -5250 2800 60  0000 L CNN
 F 1 "16Mhz" V -5150 2750 60  0000 L CNN
-F 2 "Crystal:Crystal_SMD_SeikoEpson_FA238-4Pin_3.2x2.5mm" H -5250 3050 60  0001 C CNN
+F 2 "Crystal:Crystal_SMD_7050-4Pin_7.0x5.0mm" H -5250 3050 60  0001 C CNN
 F 3 "" H -5250 3050 60  0000 C CNN
 	1    -5250 3050
@@
 TX
 $Comp
-L power:GND #PWR?
+L power:GND #PWR0135
 U 1 1 6082B89B
 P 4850 1000
-F 0 "#PWR?" H 4850 750 50  0001 C CNN
+F 0 "#PWR0135" H 4850 750 50  0001 C CNN
 F 1 "GND" H 4855 827 50  0000 C CNN
 F 2 "" H 4850 1000 50  0001 C CNN

Commit message: pre tht crystal
Parts:
- removed C2, C4: 22pF, Capacitor_SMD:C_0805_2012Metric, symbol keyboard_parts:C
- removed X1: 16Mhz, Crystal:Crystal_SMD_7050-4Pin_7.0x5.0mm, symbol keyboard_parts:XTAL
- added 16mhz1: Crystal, Crystal:Crystal_HC49-4H_Vertical, symbol Device:Crystal
Connections:
- net at U1.16 (XTAL1): now also 16mhz1.1
- net at U1.17 (XTAL2): now also 16mhz1.2
Changed lines of the file:
@@
 Wire Wire Line
 	-4200 2700 -3500 2700
-Wire Wire Line
-	-5100 3100 -3500 3100
-Wire Wire Line
-	-5100 3000 -3500 3000
-Wire Wire Line
-	-6000 3050 -6000 3350
-Connection ~ -6000 3050
-Wire Wire Line
-	-6200 3050 -6000 3050
-Wire Wire Line
-	-6000 3350 -5850 3350
-Wire Wire Line
-	-6000 2750 -6000 3050
-Wire Wire Line
-	-5850 2750 -6000 2750
-$Comp
-L keyboard_parts:C C2
-U 1 1 60849CE6
-P -5650 3350
-F 0 "C2" V -5500 3350 50  0000 C CNN
-F 1 "22pF" V -5400 3350 50  0000 C CNN
-F 2 "Capacitor_SMD:C_0805_2012Metric" H -5650 3350 60  0001 C CNN
-F 3 "" H -5650 3350 60  0000 C CNN
-	1    -5650 3350
-	0    1    1    0
-$EndComp
-$Comp
-L keyboard_parts:C C4
-U 1 1 60848A7B
-P -5650 2750
-F 0 "C4" V -5917 2750 50  0000 C CNN
-F 1 "22pF" V -5826 2750 50  0000 C CNN
-F 2 "Capacitor_SMD:C_0805_2012Metric" H -5650 2750 60  0001 C CNN
-F 3 "" H -5650 2750 60  0000 C CNN
-	1    -5650 2750
-	0    1    1    0
-$EndComp
-Wire Wire Line
-	-5100 3350 -5100 3100
-Wire Wire Line
-	-5100 3000 -5100 2750
 Text GLabel -1000 5850 0    50   Input ~ 0
 A3
@@
 	1    -3750 4550
 	1    0    0    -1
-$EndComp
-$Comp
-L power:GND #PWR0103
-U 1 1 60E5C8DE
-P -6200 3050
-F 0 "#PWR0103" H -6200 2800 50  0001 C CNN
-F 1 "GND" H -6195 2877 50  0000 C CNN
-F 2 "" H -6200 3050 50  0001 C CNN
-F 3 "" H -6200 3050 50  0001 C CNN
-	1    -6200 3050
-	0    1    1    0
 $EndComp
 $Comp
@@
 	3000 900  3000 1000
 Connection ~ 3000 1000
-Wire Wire Line
-	-5100 2750 -5250 2750
-Wire Wire Line
-	-5450 2750 -5250 2750
-Connection ~ -5250 2750
-Wire Wire Line
-	-5250 3350 -5100 3350
-Wire Wire Line
-	-5450 3350 -5250 3350
-Connection ~ -5250 3350
-$Comp
-L keyboard_parts:XTAL X1
-U 1 1 6080F4C1
-P -5250 3050
-F 0 "X1" V -5250 2800 60  0000 L CNN
-F 1 "16Mhz" V -5150 2750 60  0000 L CNN
-F 2 "Crystal:Crystal_SMD_7050-4Pin_7.0x5.0mm" H -5250 3050 60  0001 C CNN
-F 3 "" H -5250 3050 60  0000 C CNN
-	1    -5250 3050
-	0    1    1    0
-$EndComp
 Text GLabel -1000 7800 0    50   Input ~ 0
 SCK
@@
 Wire Wire Line
 	4850 1100 4850 1000
+$Comp
+L Device:Crystal 16mhz1
+U 1 1 60882EA9
+P -4950 3050
+F 0 "16mhz1" V -5000 2600 50  0000 L CNN
+F 1 "Crystal" V -4900 2600 50  0000 L CNN
+F 2 "Crystal:Crystal_HC49-4H_Vertical" H -4950 3050 50  0001 C CNN
+F 3 "~" H -4950 3050 50  0001 C CNN
+	1    -4950 3050
+	0    1    1    0
+$EndComp
+Wire Wire Line
+	-3500 3000 -4650 3000
+Wire Wire Line
+	-4650 3000 -4650 2900
+Wire Wire Line
+	-4650 2900 -4950 2900
+Wire Wire Line
+	-4950 3200 -4650 3200
+Wire Wire Line
+	-4650 3200 -4650 3100
+Wire Wire Line
+	-4650 3100 -3500 3100
 $EndSCHEMATC

Commit message: logo and updating JLB components
Parts:
- 16mhz1: symbol Device:Crystal -> monarch-rescue:Crystal-Device
- BZ1: symbol Device:Buzzer -> monarch-rescue:Buzzer-Device
- C1: symbol Device:C_Small -> monarch-rescue:C_Small-Device
- C19, C6: symbol Device:CP1_Small -> monarch-rescue:CP1_Small-Device
- C3, C5, C7, C8: symbol Device:C -> monarch-rescue:C-Device
- D1, D10, D11, D12, D13, D14, D15, D16, D17, D18, D19, D2, D20, D21, D22, D23, D24, D25, D3, D4, D5, D6, D7, D8, D9: footprint Diode_SMD:D_0805_2012Metric -> Diode_SMD:D_SOD-123; symbol Device:D -> monarch-rescue:D-Device
- D26, D27, RED1: symbol Device:LED -> monarch-rescue:LED-Device
- J1, J2: symbol Connector:USB_C_Receptacle_USB2.0 -> monarch-rescue:USB_C_Receptacle_USB2.0-Connector
- JP1: symbol Device:Jumper -> monarch-rescue:Jumper-Device
- R1, R2, R3, R4, R5, R7: symbol Device:R_US -> monarch-rescue:R_US-Device
- R6, R8: symbol Device:R_Small_US -> monarch-rescue:R_Small_US-Device
- SW19: symbol Device:Rotary_Encoder_Switch -> monarch-rescue:Rotary_Encoder_Switch-Device
- U2: symbol Regulator_Linear:MIC5219-5.0YMM -> monarch-rescue:MIC5219-5.0YMM-Regulator_Linear
