File: monarch.kicad_pcb (KiCad board)
At the start: 2 copper layers, 165.4 x 129.6 mm, 142 parts, among them J1 USB_C_Receptacle_USB2.0, J2 USB_C_Receptacle_USB2.0, J3 OLED, SW1 SW_PUSH, SW10 SW_PUSH, SW11 SW_PUSH, SW12 SW_PUSH, SW13 SW_PUSH, SW14 SW_PUSH, SW15 SW_PUSH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

Commit message: left side completed
Parts:
- added H9: Hole, MountingHole:MountingHole_2.2mm_M2, F.Cu at (174.1, 95.8)
- moved R4 11.2 mm to (38.3, 15.3), turned to 90 degrees
- moved J1 7.71 mm to (28.8, 14.6)
- moved R3 6.24 mm to (28.0, 19.7), turned to 90 degrees
- moved G*** 4.99 mm to (36.6, 25.0)
- moved J2 2.66 mm to (162.5, 97.3)
- moved H1 0.68 mm to (126.0, 12.4)
- moved H2 0.59 mm to (156.0, 86.6)
- moved L6 0.51 mm to (166.1, 103.7)
- moved H1 0.07 mm to (132.0, 13.6)
Routing:
- net UVCC: track 195.3 -> 184.8 mm
- net Net-(J1-PadB5): track 2.23 -> 7.76 mm, vias 0 -> 1
- net Net-(J1-PadA5): track 10.7 -> 5.25 mm, vias 2 -> 0
- net GND: track 205.8 -> 203.2 mm, vias 26 -> 28
- net VCC: track 974.7 -> 972.3 mm, vias 23 -> 22
- net Net-(J1-PadA7): track 151.0 -> 153.0 mm
- net Net-(J1-PadA6): track 156.1 -> 158.0 mm
- net Net-(L33-Pad1): track 58.1 -> 56.3 mm
- net RX: track 41.2 -> 39.5 mm
- net Net-(L35-Pad1): track 13.8 -> 12.5 mm
- net COL1: track 207.6 -> 206.6 mm
- net Net-(L6-Pad1): track 33.2 -> 33.8 mm
- net Net-(L36-Pad1): track 11.1 -> 10.9 mm, vias 2 -> 0
